File: tmp-seq-one/seq-one-control-board/seq-one-control-board.kicad_sch (KiCad schematic)
At the start: 46 parts, among them J1 Step Button, J10 Signals, J11 Power, J2 Step Jack, J3 Start Button, J4 Start Jack, J5 Reset Button, J6 Reset Jack, J7 Loop Switch, J8 OneTwo Switch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

Commit message: Updating to KiCad 9.0
Parts:
- added C11: C, symbol Device:C
- added R13: R, symbol Device:R
- R12: value 470 -> 1K
Connections:
- net +12V: now also R12.2
- net GND: now also C11.2; no longer R12.2, U2.11, U2.12, U2.13
- net ~STEP_ACTIVE: now also U2.11, U2.12, U2.13; no longer D7.2 (A)
- net at U2.10: now also D7.1 (K)
- net at R12.1: now also D7.2 (A); no longer D7.1 (K)
- net at U1.3: now also C11.1, R13.2; no longer U1.6
- new net: R13.1, U1.6
- no-connect marks 1 -> 0
Other:
- note added: "FIXME: Button Debouncing"
- note added: "FIXME: Debounce here? Or at the diodes?"
- note added: "FIXME: Note here which way the switches work"
- note added: "FIXME: ~STEP_ACTIVE doesn't pull up high enough to activate the logic for the step outs"
- note removed: "FIXME: Buffer Needed?"
- moved on the sheet: D7, R12, U2C
