File: train-set-building-light/train-set-building-light.kicad_pcb (KiCad board)
At the start: 2 copper layers, 127 x 14 mm, 54 parts

Commit message: Updating to KiCad 9.0
Other:
- net class Default removed
